File: NPK_smd.kicad_pcb (KiCad board)
At the start: 2 copper layers, 64.2 x 85.9 mm, 58 parts, among them J2 Screw_Terminal_01x04, J3 USB_C_Receptacle_USB2.0_16P, Q3 SS8050, Q4 SS8050, SW1 SW_Push, SW2 SW_Push, SW3 SW_SPST, U1 AMS1117-3.3, U2 MAX485ESA_T, U3 LM2596S-ADJ, U4 ESP32-WROOM-32, U6 USBLC6-2SC6, U7 CH340C

Commit message: updated
Parts:
- added J1: DHT, Connector_PinSocket_2.54mm:PinSocket_1x03_P2.54mm_Vertical, F.Cu at (177.2, 88.5)
- moved JP1 1.90 mm to (119.8, 70.6)
- moved D1 1.38 mm to (114.0, 71.0)
Connections:
- U4 pad 33: unconnected-(U4-IO21-Pad33) -> /DHT
Routing:
- net /WS28: track 42.4 -> 40.9 mm
- net Net-(D1-VDD): track 8.27 -> 9.05 mm

Commit message: updated
Parts:
- moved J1 51.2 mm to (150.7, 44.8), turned to -90 degrees
Connections:
- U4 pad 11: unconnected-(U4-IO26-Pad11) -> /DHT
- U4 pad 33: /DHT -> unconnected-(U4-IO21-Pad33)
Routing:
- net /DHT: track 0.00 -> 8.01 mm, vias 0 -> 1
Changed lines of the file:
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@@
 	(net 58 "unconnected-(U4-IO27-Pad12)")
 	(net 59 "unconnected-(U4-SENSOR_VN-Pad5)")
-	(net 60 "unconnected-(U4-IO26-Pad11)")
+	(net 60 "unconnected-(U4-IO21-Pad33)")
 	(net 61 "unconnected-(U4-IO33-Pad9)")
 	(net 62 "unconnected-(U4-IO25-Pad10)")
@@
 			(size 1.5 0.9)
 			(layers "F.Cu" "F.Mask" "F.Paste")
-			(net 60 "unconnected-(U4-IO26-Pad11)")
+			(net 39 "/DHT")
 			(pinfunction "IO26")
-			(pintype "bidirectional+no_connect")
+			(pintype "bidirectional")
 		)
 		(pad "12" smd rect
@@
 			(size 1.5 0.9)
 			(layers "F.Cu" "F.Mask" "F.Paste")
-			(net 39 "/DHT")
+			(net 60 "unconnected-(U4-IO21-Pad33)")
 			(pinfunction "IO21")
-			(pintype "bidirectional")
+			(pintype "bidirectional+no_connect")
 		)
 		(pad "34" smd rect
@@
 	(footprint "Connector_PinSocket_2.54mm:PinSocket_1x03_P2.54mm_Vertical"
 		(layer "F.Cu")
-		(at 177.175 88.5 180)
+		(at 150.665 44.75 -90)
 		(descr "Through hole straight socket strip, 1x03, 2.54mm pitch, single row (from Kicad 4.0.7), script generated")
 		(tags "Through hole socket strip THT 1x03 2.54mm single row")
 		(property "Reference" "J1"
-			(at 0 -2.77 0)
+			(at 0 -2.77 90)
 			(layer "F.SilkS")
 			(effects
@@
 		)
 		(property "Value" "DHT"
-			(at 0 7.85 0)
+			(at 0 7.85 90)
 			(layer "F.Fab")
 			(effects
@@
 		)
 		(property "Datasheet" "~"
-			(at 0 0 0)
+			(at 0 0 90)
 			(layer "F.Fab")
 			(hide yes)
@@
 		)
 		(property "Description" "Generic connector, single row, 01x03, script generated"
-			(at 0 0 0)
+			(at 0 0 90)
 			(layer "F.Fab")
 			(hide yes)
@@
 		(attr through_hole)
 		(fp_line
-			(start 1.33 1.27)
+			(start -1.33 6.41)
 			(end 1.33 6.41)
 			(stroke
@@
 		)
 		(fp_line
-			(start 1.33 -1.33)
-			(end 1.33 0)
+			(start -1.33 1.27)
+			(end -1.33 6.41)
 			(stroke
 				(width 0.12)
@@
 		)
 		(fp_line
-			(start 0 -1.33)
-			(end 1.33 -1.33)
+			(start -1.33 1.27)
+			(end 1.33 1.27)
 			(stroke
 				(width 0.12)
@@
 		)
 		(fp_line
-			(start -1.33 6.41)
+			(start 1.33 1.27)
 			(end 1.33 6.41)
 			(stroke
@@
 		)
 		(fp_line
-			(start -1.33 1.27)
-			(end 1.33 1.27)
+			(start 0 -1.33)
+			(end 1.33 -1.33)
 			(stroke
 				(width 0.12)
@@
 		)
 		(fp_line
-			(start -1.33 1.27)
-			(end -1.33 6.41)
+			(start 1.33 -1.33)
+			(end 1.33 0)
 			(stroke
 				(width 0.12)
@@
 		)
 		(fp_line
-			(start 1.75 6.85)
-			(end -1.8 6.85)
+			(start -1.8 6.85)
+			(end -1.8 -1.8)
 			(stroke
 				(width 0.05)
@@
 		)
 		(fp_line
-			(start 1.75 -1.8)
-			(end 1.75 6.85)
+			(start 1.75 6.85)
+			(end -1.8 6.85)
 			(stroke
 				(width 0.05)
@@
 		)
 		(fp_line
-			(start -1.8 6.85)
-			(end -1.8 -1.8)
+			(start -1.8 -1.8)
+			(end 1.75 -1.8)
 			(stroke
 				(width 0.05)
@@
 		)
 		(fp_line
-			(start -1.8 -1.8)
-			(end 1.75 -1.8)
+			(start 1.75 -1.8)
+			(end 1.75 6.85)
 			(stroke
 				(width 0.05)
@@
 		)
 		(fp_line
-			(start 1.27 6.35)
-			(end -1.27 6.35)
+			(start -1.27 6.35)
+			(end -1.27 -1.27)
 			(stroke
 				(width 0.1)
@@
 		)
 		(fp_line
-			(start 1.27 -0.635)
-			(end 1.27 6.35)
+			(start 1.27 6.35)
+			(end -1.27 6.35)
 			(stroke
 				(width 0.1)
@@
 		)
 		(fp_line
-			(start 0.635 -1.27)
-			(end 1.27 -0.635)
+			(start 1.27 -0.635)
+			(end 1.27 6.35)
 			(stroke
 				(width 0.1)
@@
 		)
 		(fp_line
-			(start -1.27 6.35)
-			(end -1.27 -1.27)
+			(start -1.27 -1.27)
+			(end 0.635 -1.27)
 			(stroke
 				(width 0.1)
@@
 		)
 		(fp_line
-			(start -1.27 -1.27)
-			(end 0.635 -1.27)
+			(start 0.635 -1.27)
+			(end 1.27 -0.635)
 			(stroke
 				(width 0.1)
@@
 		)
 		(fp_text user "${REFERENCE}"
-			(at 0 2.54 90)
+			(at 0 2.54 0)
 			(layer "F.Fab")
 			(effects
@@
 		)
 		(pad "1" thru_hole rect
-			(at 0 0 180)
+			(at 0 0 270)
 			(size 1.7 1.7)
 			(drill 1)
@@
 		)
 		(pad "2" thru_hole circle
-			(at 0 2.54 180)
+			(at 0 2.54 270)
 			(size 1.7 1.7)
 			(drill 1)
@@
 		)
 		(pad "3" thru_hole circle
-			(at 0 5.08 180)
+			(at 0 5.08 270)
 			(size 1.7 1.7)
 			(drill 1)
@@
 		(net 34)
 	)
+	(via
+		(at 151.46 51.375)
+		(size 0.6)
+		(drill 0.3)
+		(layers "F.Cu" "B.Cu")
+		(net 39)
+	)
+	(segment
+		(start 148.125 45.8)
+		(end 151.46 49.135)
+		(width 0.2)
+		(layer "B.Cu")
+		(net 39)
+	)
+	(segment
+		(start 148.125 44.75)
+		(end 148.125 45.8)
+		(width 0.2)
+		(layer "B.Cu")
+		(net 39)
+	)
+	(segment
+		(start 151.46 49.135)
+		(end 151.46 51.375)
+		(width 0.2)
+		(layer "B.Cu")
+		(net 39)
+	)
 	(segment

Commit message: size minimizations and updations
Parts:
- removed BT2: BK-18650-PC6, 18650-3cell holder:BAT_BK-18650-PC6
- removed JP1: Jumper_3_Open, PCM_SparkFun-Jumper:Jumper_3_NO
- removed U5: ~, custom:BMS-10A-3S
- added G***: LOGO, LOGO, B.Cu at (130.1, 87.3)
- added G***: LOGO, LOGO, B.Cu at (106.3, 60.2)
- added J4: Conn_01x02_Pin, custom:solder-pad, F.Cu at (104.9, 88.3)
- added REF**: ESD-Logo_6.6x6mm_SilkScreen, Symbol:ESD-Logo_6.6x6mm_SilkScreen, B.Cu at (106.0, 69.3)
- C3, C4, D2, D4, Q3, Q4, R1, R11, R12, R13, R14, R15, R16, R17, R18, R19, R2, R20, R21, R3, R4, R5, R6, R7, U2: moved to B.Cu
- SW1, SW2: footprint Button_Switch_SMD:SW_Tactile_SPST_NO_Straight_CK_PTS636Sx25SMTRLFS -> tactile-switch:SW_B3U-1000PM
- moved J1 51.6 mm to (108.8, 75.0)
- moved SW3 50.6 mm to (115.0, 94.8), turned to 90 degrees
- moved J2 50.3 mm to (111.2, 93.7)
- moved BZ1 48.0 mm to (117.9, 67.4), turned to -90 degrees
- moved R15 37.4 mm to (120.6, 70.3), turned to 90 degrees
- moved R4 37.2 mm to (127.5, 50.3), turned to 0 degrees
- moved R14 36.4 mm to (120.8, 75.6), turned to -90 degrees
- moved D4 35.2 mm to (125.3, 74.7), turned to 180 degrees
- moved R13 32.2 mm to (123.8, 69.8), turned to 90 degrees
- moved R12 31.0 mm to (126.7, 70.2), turned to 90 degrees
- moved D3 28.7 mm to (134.5, 44.8)
- moved R1 27.9 mm to (127.5, 53.3), turned to 0 degrees
- moved R6 26.9 mm to (130.6, 43.5), turned to 90 degrees
- moved 100uf1 26.2 mm to (138.7, 43.2)
- moved R20 25.8 mm to (138.7, 60.9), turned to -90 degrees
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Connections:
- D1 pad 1: Net-(D1-VDD) -> 3V3
- U4 pad 11: /DHT -> unconnected-(U4-IO26-Pad11)
- U4 pad 26: /buz -> /WS28
- U4 pad 30: /WS28 -> /buz
- U4 pad 31: unconnected-(U4-IO19-Pad31) -> /DHT
Routing:
- net /B2: track 95.0 -> 0.00 mm, vias 4 -> 0
- net /B1: track 81.7 -> 0.00 mm, vias 8 -> 0
- net /12V: track 95.8 -> 35.1 mm, vias 0 -> 1
- net 5V: track 167.1 -> 130.0 mm, vias 10 -> 6
- net ESP32_EN: track 53.9 -> 27.0 mm, vias 2 -> 4
- net /DHT: track 8.01 -> 34.7 mm, vias 1 -> 2
- net GND: track 62.5 -> 37.2 mm, vias 75 -> 44
- net /IO23: track 30.9 -> 11.7 mm, vias 2 -> 1
- net 3V3: track 5.56 -> 24.4 mm, vias 0 -> 4
- net /WS28: track 40.9 -> 22.4 mm
- net /IO22: track 25.2 -> 7.28 mm, vias 2 -> 1
- net Net-(U7-TXD): track 41.8 -> 28.0 mm, vias 2 -> 3
- net /IO13: track 33.6 -> 22.0 mm, vias 2 -> 1
- net Net-(U7-RXD): track 46.3 -> 34.8 mm, vias 2 -> 3
- net /buz: track 27.7 -> 16.3 mm
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Other:
- board size 64.2 x 85.9 mm -> 50.3 x 58 mm
- board text added: "+12V"
- board text added: "12V"
- board text added: "A"
- board text added: "B"
- board text added: "DHT"
- board text added: "G"

Commit message: version-1.0 rev 2026-04-11
Parts:
- removed REF**: ESD-Logo_6.6x6mm_SilkScreen, Symbol:ESD-Logo_6.6x6mm_SilkScreen
- removed SW3: SW_SPST, TestPoint:TestPoint_2Pads_Pitch2.54mm_Drill0.8mm
- added G***: LOGO, LOGO, F.Cu at (117.5, 55.6)
- added J5: prog, Connector_PinHeader_2.54mm:PinHeader_1x04_P2.54mm_Vertical_SMD_Pin1Left, F.Cu at (133.7, 71.1)
- added SW4: SW_Push, tactile-switch:SW_B3U-1000PM, F.Cu at (126.8, 42.3)
- C1, C12, C2, CP1, CP2, U1, U7: moved to B.Cu
- R19, R20, R6: moved to F.Cu
- moved R19 32.9 mm to (108.4, 62.3), turned to 180 degrees
- moved R20 30.4 mm to (108.3, 59.7), turned to 0 degrees
- moved R21 30.1 mm to (106.4, 65.1), turned to 0 degrees
- moved U1 18.4 mm to (138.1, 89.7), turned to -90 degrees
- moved C1 15.2 mm to (143.6, 85.9), turned to 90 degrees
- moved CP1 15.0 mm to (146.0, 85.9), turned to -90 degrees
- moved C2 14.0 mm to (132.7, 82.4), turned to -90 degrees
- moved C12 12.6 mm to (101.8, 59.7)
- moved CP2 11.0 mm to (135.4, 82.4)
- moved G*** 9.69 mm to (107.2, 50.6), turned to -90 degrees
- moved SW1 6.66 mm to (115.0, 42.5), turned to 0 degrees
- moved SW2 5.85 mm to (121.3, 42.4)
- moved G*** 5.68 mm to (124.7, 89.0), turned to 180 degrees
- moved D1 1.67 mm to (107.1, 68.6), turned to 180 degrees
- moved J1 1.30 mm to (109.9, 74.2)
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Connections:
- U4 pad 12: unconnected-(U4-IO27-Pad12) -> /user
- U4 pad 23: ADC2_3/TCH3 -> unconnected-(U4-IO15-Pad23)
- U4 pad 26: /WS28 -> /DHT
- U4 pad 27: unconnected-(U4-IO16-Pad27) -> /WS28
- U4 pad 31: /DHT -> unconnected-(U4-IO19-Pad31)
Routing:
- net PRG_RX: track 2.48 -> 39.5 mm
- net PRG_TX: track 5.48 -> 37.8 mm, vias 1 -> 2
- net Net-(U7-RXD): track 34.8 -> 2.69 mm, vias 3 -> 1
- net Net-(U7-TXD): track 28.0 -> 7.88 mm, vias 3 -> 2
- net 5V: track 130.0 -> 118.2 mm, vias 6 -> 9
- net /DHT: track 34.7 -> 23.9 mm, vias 2 -> 3
- net GND: track 37.2 -> 30.2 mm
- net Net-(Q4-E): track 19.4 -> 25.9 mm, vias 1 -> 2
- net /user: track 0.00 -> 6.01 mm, vias 0 -> 2
- net /WS28: track 22.4 -> 25.6 mm
- net ESP32_EN: track 27.0 -> 29.9 mm, vias 4 -> 2
- net /D+: track 13.3 -> 15.6 mm, vias 0 -> 1
- net Net-(Q3-E): track 26.4 -> 27.9 mm, vias 3 -> 2
- net /buz: track 16.3 -> 15.0 mm
- net Net-(Q3-B): track 7.80 -> 8.63 mm, vias 0 -> 2
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Other:
- board size 50.3 x 58 mm -> 50.3 x 58.3 mm
- board text added: "Bhoomitra"
- board text added: "LED"
- board text added: "PROG"
- board text added: "Rev-04/26"
- board text added: "Ver-1.0"
- board text added: "by AR RoboTics"
- board text removed: "+12V"
