File: NPK_smd.kicad_sch (KiCad schematic)
At the start: 58 parts, among them J2 Screw_Terminal_01x04, J3 USB_C_Receptacle_USB2.0_16P, Q3 SS8050, Q4 SS8050, SW1 SW_Push, SW2 SW_Push, SW3 SW_SPST, U1 AMS1117-3.3, U2 MAX485ESA_T, U3 LM2596S-ADJ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

Commit message: updated
Parts:
- added J1: DHT, Connector_PinSocket_2.54mm:PinSocket_1x03_P2.54mm_Vertical, symbol Connector:Conn_01x03_Pin
Connections:
- net 3V3: now also J1.1 (Pin_1)
- net GND: now also J1.3 (Pin_3)
- net DHT: now reaches U4.33 (IO21)
- net DHT: now also J1.2 (Pin_2)
- no-connect marks 28 -> 27
Other:
- moved on the sheet: BT2, BZ1, D4, J2, R11, R14, R15, R16, R19, R8, SW1, SW2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

Commit message: updated
Connections:
- net DHT: now also U4.11 (IO26); no longer U4.33 (IO21)
Changed lines of the file:
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@@
+	)
+	(no_connect
+		(at 227.33 86.36)
 	)
 	(no_connect
@@
 	)
 	(no_connect
-		(at 227.33 96.52)
-	)
-	(no_connect
 		(at 196.85 58.42)
 	)
@@
 	(wire
 		(pts
-			(xy 227.33 86.36) (xy 233.68 86.36)
-		)
-		(stroke
-			(width 0)
-			(type default)
-		)
-	)
-	(wire
-		(pts
 			(xy 156.21 74.93) (xy 156.21 71.12)
 		)
@@
 		(pts
 			(xy 147.32 147.32) (xy 149.86 147.32)
+		)
+		(stroke
+			(width 0)
+			(type default)
+		)
+	)
+	(wire
+		(pts
+			(xy 232.41 96.52) (xy 227.33 96.52)
 		)
 		(stroke
@@
 		)
 	)
-	(label "DHT"
-		(at 233.68 86.36 180)
-		(effects
-			(font
-				(size 1.27 1.27)
-			)
-			(justify right bottom)
-		)
-	)
 	(label "D-"
 		(at 67.31 43.18 0)
@@
 		)
 	)
+	(label "DHT"
+		(at 232.41 96.52 180)
+		(effects
+			(font
+				(size 1.27 1.27)
+			)
+			(justify right bottom)
+		)
+	)

Commit message: size minimizations and updations
Parts:
- removed BT2: BK-18650-PC6, 18650-3cell holder:BAT_BK-18650-PC6, symbol 18650-3cell:BK-18650-PC6
- removed JP1: Jumper_3_Open, PCM_SparkFun-Jumper:Jumper_3_NO, symbol Jumper:Jumper_3_Open
- removed U5: ~, custom:BMS-10A-3S, symbol custom_symbols:bms
- added J4: Conn_01x02_Pin, custom:solder-pad, symbol Connector:Conn_01x02_Pin
- SW1, SW2: footprint Button_Switch_SMD:SW_Tactile_SPST_NO_Straight_CK_PTS636Sx25SMTRLFS -> tactile-switch:SW_B3U-1000PM
Connections:
- net 12V: now also J4.2 (Pin_2)
- net 3V3: now also D1.1 (VDD)
- net DHT: no longer U4.11 (IO26)
- net GND: now also J4.1 (Pin_1)
- net WS28: now also U4.26 (IO4); no longer U4.30 (IO18)
- net buz: now also U4.30 (IO18); no longer U4.26 (IO4)
- net ADC2_3/TCH3: no longer names the net of U4.23 (IO15)
- no-connect marks 27 -> 29

Commit message: version-1.0 rev 2026-04-11
Parts:
- removed SW3: SW_SPST, TestPoint:TestPoint_2Pads_Pitch2.54mm_Drill0.8mm, symbol Switch:SW_SPST
- added J5: prog, Connector_PinHeader_2.54mm:PinHeader_1x04_P2.54mm_Vertical_SMD_Pin1Left, symbol Connector:Conn_01x04_Pin
- added SW4: SW_Push, tactile-switch:SW_B3U-1000PM, symbol Switch:SW_Push
Connections:
- net 3V3: now also J5.3 (Pin_3)
- net DHT: now also U4.26 (IO4)
- net GND: now also J5.4 (Pin_4), SW4.1
- net PRG_RX: now also J5.2 (Pin_2)
- net PRG_TX: now also J5.1 (Pin_1)
- net WS28: now also U4.27 (IO16); no longer U4.26 (IO4)
- net user: now reaches U4.12 (IO27)
- net user: now also SW4.2
- no-connect marks 29 -> 27
Other:
- note removed: "3V3-LDO"
- note removed: "Boot/En-SW"
- note removed: "ESP32"
- note removed: "LEDS"
- note removed: "TypeC-Uart"
- company: (none) -> AR RoboTics
- title: (none) -> Bhoomitra
- moved on the sheet: 100uf1, BZ1, C3, C4, C6, D1, D2, D3, D4, J1, J2, J4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
